File: maciifxsimm.kicad_pcb (KiCad board)
At the start: 2 copper layers, 97.8 x 22.2 mm, 11 parts, among them J1 SIMM64_EDGE, U1 KM41C16000CK, U2 KM41C16000CK, U3 KM41C16000CK, U4 KM41C16000CK, U5 KM41C16000CK, U6 KM41C16000CK, U7 KM41C16000CK, U8 KM41C16000CK

Commit message: v1 sent to fab
Routing:
- net GND: track 2.48 -> 17.4 mm, vias 69 -> 71
Other:
- board text added: "JLCJLCJLCJLC"
- board text added: "Macintosh IIfx 16 MB SIMM (v1) https://github.com/hanshuebner/maciifxsimm"
- board text removed: "KEEP RETROCOMPUTING AFFORDABLE!"
- board text removed: "Macintosh IIfx 16 MB SIMM"
- board text removed: "© 2019 TUBETIMEUS © 2023 Hans Hübner"
Changed lines of the file:
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@@
   (gr_arc (start 103.9495 82.55) (mid 105.072032 83.014968) (end 105.537 84.1375)
     (stroke (width 0.05) (type solid)) (layer "Edge.Cuts"))
-  (gr_text "Macintosh IIfx 16 MB SIMM" (at 152.4 69.469) (layer "B.SilkS")
+  (gr_text "Macintosh IIfx 16 MB SIMM (v1)\nhttps://github.com/hanshuebner/maciifxsimm" (at 152.4 69.469) (layer "B.SilkS")
     (effects (font (size 1.27 1.27) (thickness 0.15)) (justify mirror))
   )
-  (gr_text "© 2019 TUBETIMEUS\n© 2023 Hans Hübner" (at 152.4 79.756) (layer "B.SilkS")
-    (effects (font (size 1.27 1.27) (thickness 0.1524)) (justify mirror))
-  )
-  (gr_text "KEEP RETROCOMPUTING AFFORDABLE!" (at 151.765 83.566) (layer "B.SilkS")
-    (effects (font (size 1.27 1.27) (thickness 0.15)) (justify mirror))
+  (gr_text "JLCJLCJLCJLC" (at 114.173 80.645 90) (layer "F.SilkS")
+    (effects (font (size 1 1) (thickness 0.15)) (justify left bottom))
   )
   (dimension (type aligned) (layer "Dwgs.User")
@@
   (via (at 135.636 71.882) (size 0.5) (drill 0.3) (layers "F.Cu" "B.Cu") (free) (net 1))
   (via (at 181.229 83.312) (size 0.5) (drill 0.3) (layers "F.Cu" "B.Cu") (free) (net 1))
+  (via (at 170.815 83.439) (size 0.8) (drill 0.5) (layers "F.Cu" "B.Cu") (net 1))
   (via (at 135.636 73.152) (size 0.5) (drill 0.3) (layers "F.Cu" "B.Cu") (free) (net 1))
   (via (at 180.086 71.882) (size 0.5) (drill 0.3) (layers "F.Cu" "B.Cu") (free) (net 1))
@@
   (via (at 156.972 70.612) (size 0.5) (drill 0.3) (layers "F.Cu" "B.Cu") (free) (net 1))
   (via (at 135.636 70.612) (size 0.5) (drill 0.3) (layers "F.Cu" "B.Cu") (free) (net 1))
+  (via (at 194.945 84.328) (size 0.8) (drill 0.5) (layers "F.Cu" "B.Cu") (net 1))
   (via (at 172.72 84.582) (size 0.5) (drill 0.3) (layers "F.Cu" "B.Cu") (free) (net 1))
   (via (at 125.222 70.612) (size 0.5) (drill 0.3) (layers "F.Cu" "B.Cu") (free) (net 1))
@@
   (via (at 183.769 84.582) (size 0.5) (drill 0.3) (layers "F.Cu" "B.Cu") (free) (net 1))
   (segment (start 163.195 82.677) (end 161.798 84.074) (width 0.127) (layer "B.Cu") (net 1))
+  (segment (start 170.815 86.36) (end 170.815 83.439) (width 0.508) (layer "B.Cu") (net 1))
+  (segment (start 132.715 83.693) (end 132.334 83.312) (width 0.508) (layer "B.Cu") (net 1))
+  (segment (start 109.855 86.36) (end 109.855 83.947) (width 0.508) (layer "B.Cu") (net 1))
+  (segment (start 131.445 84.201) (end 132.334 83.312) (width 0.508) (layer "B.Cu") (net 1))
+  (segment (start 131.445 86.36) (end 131.445 84.201) (width 0.508) (layer "B.Cu") (net 1))
   (segment (start 161.798 84.074) (end 161.798 84.582) (width 0.127) (layer "B.Cu") (net 1))
+  (segment (start 194.945 86.36) (end 194.945 84.328) (width 0.508) (layer "B.Cu") (net 1))
+  (segment (start 132.715 86.36) (end 132.715 83.693) (width 0.508) (layer "B.Cu") (net 1))
+  (segment (start 109.855 83.947) (end 110.49 83.312) (width 0.508) (layer "B.Cu") (net 1))
   (segment (start 175.5295 79.0115) (end 176.02 79.502) (width 0.127) (layer "F.Cu") (net 2))
   (segment (start 132.8245 79.0115) (end 142.7655 79.0115) (width 0.127) (layer "F.Cu") (net 2))
