File: maciifxsimm.kicad_pcb (KiCad board)
At the start: 2 copper layers, 97.8 x 22.2 mm, 19 parts, among them J1 SIMM64_EDGE, U1 KM41C16000CK, U2 KM41C16000CK, U3 KM41C16000CK, U4 KM41C16000CK, U5 KM41C16000CK, U6 KM41C16000CK, U7 KM41C16000CK, U8 KM41C16000CK

Commit message: Add files via upload
4-layer modifications
Parts:
- moved C1 10.3 mm to (113.9, 75.9), turned to 180 degrees
- moved C3 10.2 mm to (135.9, 75.9), turned to 180 degrees
- moved C2 10.1 mm to (125.1, 75.9), turned to 180 degrees
- moved C5 10.1 mm to (157.9, 75.9), turned to 180 degrees
- moved C4 10.1 mm to (147.0, 75.9), turned to 180 degrees
- moved C6 10.1 mm to (168.9, 75.9), turned to 180 degrees
- moved C7 9.78 mm to (179.9, 76.0), turned to 180 degrees
- moved C8 9.54 mm to (190.9, 75.9), turned to 180 degrees
- moved U1 0.29 mm to (114.0, 75.7)
Connections:
- J1 pad 10: (no net) -> GND
- J1 pad 24: (no net) -> GND
- J1 pad 30: (no net) -> GND
- J1 pad 36: (no net) -> GND
- J1 pad 49: (no net) -> GND
- J1 pad 54: (no net) -> GND
- J1 pad 56: (no net) -> GND
Routing:
- net GND: track 14.9 -> 301.3 mm, vias 61 -> 24
- net VCC: track 240.2 -> 480.4 mm
- net A11: track 90.2 -> 109.1 mm, vias 1 -> 8
- net A7: track 92.8 -> 110.8 mm, vias 1 -> 8
- net ~{CAS}: track 86.7 -> 104.4 mm, vias 1 -> 8
- net ~{RAS}: track 88.4 -> 105.9 mm, vias 1 -> 8
- net A3: track 96.9 -> 114.0 mm, vias 1 -> 8
- net A0: track 93.6 -> 109.8 mm, vias 1 -> 8
- net A2: track 96.4 -> 112.3 mm, vias 1 -> 8
- net A1: track 95.7 -> 111.4 mm, vias 1 -> 8
- net A10: track 92.1 -> 107.7 mm, vias 1 -> 8
- net A9: track 90.2 -> 105.7 mm, vias 1 -> 8
- net A5: track 96.4 -> 111.6 mm, vias 1 -> 8
- net A8: track 91.5 -> 105.3 mm, vias 1 -> 8
- net A4: track 96.8 -> 110.4 mm, vias 1 -> 8
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- added copper zone on In1.Cu, net GND
- added copper zone on In2.Cu, net VCC
- removed copper zone on B.Cu, net GND
- removed copper zone on F.Cu, net GND
Other:
- copper layers 2 -> 4
- rule pad_to_mask_clearance: 0.051 -> 0
- board text removed: "Macintosh IIfx 16 MB SIMM (v2) https://github.com/hanshuebner/maciifxsimm"
